Commit message: Version 2; cleanup

File: config/telescope.srdf.xacro (robot description, xacro)
@@ -7,11 +7,13 @@
     <joint name="el_joint" value="1.57" />
     <joint name="az_joint" value="1.57" />
+    <joint name="eef_joint" value="0.0" />
   </group_state>
   <group_state name="zenith" group="telgroup">
     <joint name="el_joint" value="0.0" />
     <joint name="az_joint" value="1.57" />
+    <joint name="eef_joint" value="0.0" />
   </group_state>
   <virtual_joint name="virtual_joint" type="floating" parent_frame="world" child_link="base_link" />
-  <end_effector name="eef_link" parent_link="el_link" group="telgroup" parent_group="telgroup"/>
+  <end_effector name="eef_link" parent_link="el_link" group="telgroup" parent_group=""/>
     <disable_collisions link1="azimuth_link" link2="base_link" reason="Never"/>
     <disable_collisions link1="azimuth_link" link2="base_link2" reason="Adjacent"/>

Commit message: Version 4; update to urdf

File: config/telescope.srdf.xacro (robot description, xacro)
@@ -4,7 +4,12 @@
         <chain base_link="base_link" tip_link="eef_link"/>
   </group>
+  <group_state name="point" group="telgroup">
+    <joint name="az_joint" value="0.524" />
+    <joint name="el_joint" value="0.8425" />
+    <joint name="eef_joint" value="0.0" />
+  </group_state>
   <group_state name="park" group="telgroup">
-    <joint name="el_joint" value="1.57" />
-    <joint name="az_joint" value="1.57" />
+    <joint name="az_joint" value="1.569" />
+    <joint name="el_joint" value="-1.569" />
     <joint name="eef_joint" value="0.0" />
   </group_state>
@@ -16,13 +21,13 @@
   <virtual_joint name="virtual_joint" type="floating" parent_frame="world" child_link="base_link" />
   <end_effector name="eef_link" parent_link="el_link" group="telgroup" parent_group=""/>
-    <disable_collisions link1="azimuth_link" link2="base_link" reason="Never"/>
-    <disable_collisions link1="azimuth_link" link2="base_link2" reason="Adjacent"/>
-    <disable_collisions link1="azimuth_link" link2="el_dummy" reason="Never"/>
-    <disable_collisions link1="azimuth_link" link2="el_link" reason="Adjacent"/>
+    <disable_collisions link1="azimuth_bracket" link2="azimuth_servo" reason="Adjacent"/>
+    <disable_collisions link1="azimuth_bracket" link2="base_link" reason="Never"/>
+    <disable_collisions link1="azimuth_bracket" link2="base_link2" reason="Adjacent"/>
+    <disable_collisions link1="azimuth_servo" link2="base_link" reason="Never"/>
+    <disable_collisions link1="azimuth_servo" link2="base_link2" reason="Never"/>
+    <disable_collisions link1="azimuth_servo" link2="el_link" reason="Adjacent"/>
     <disable_collisions link1="base_link" link2="base_link2" reason="Adjacent"/>
-    <disable_collisions link1="base_link" link2="el_dummy" reason="Never"/>
     <disable_collisions link1="base_link" link2="el_link" reason="Never"/>
-    <disable_collisions link1="base_link2" link2="el_dummy" reason="Never"/>
     <disable_collisions link1="base_link2" link2="el_link" reason="Never"/>
-    <disable_collisions link1="el_dummy" link2="el_link" reason="Adjacent"/>
+    <disable_collisions link1="azimuth_bracket" link2="el_link" reason="Never"/>
 </robot>

File: config/urdf/tel.urdf (robot description, URDF)
Before this commit: robot telescope, 6 links, 5 joints
Links:
- removed link azimuth_link
- removed link el_dummy
- added link azimuth_bracket; collision mesh filename=package://robotic_telescope/config/urdf/meshes/multi_functi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 scale=0.005 0.005 0.005; visual mesh filename=package://robotic_telescope/config/urdf/meshes/multi_functi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 scale=0.005 0.005 0.005
- added link azimuth_servo; collision mesh filename=package://robotic_telescope/config/urdf/meshes/mg996r_servo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 scale=0.005 0.005 0.005; visual mesh filename=package://robotic_telescope/config/urdf/meshes/mg996r_servo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 scale=0.005 0.005 0.005
- link el_link: geometry collision mesh filename=package://robotic_telescope/config/urdf/meshes/u_bracket.stl scale=0.0004 0.0004 0.0004; visual mesh filename=package://robotic_telescope/config/urdf/meshes/u_bracket.stl scale=0.0004 0.0004 0.0004
Joints:
- removed joint el_dummy_joint
- added joint azimuth_servo_joint_dummy: type fixed, parent azimuth_bracket, child azimuth_servo, origin xyz=0.0 0 0.0 rpy=0 0 0, axis 0 0 0
- joint az_joint: axis 0 0 1 -> 1 0 0; child azimuth_link -> azimuth_bracket; origin xyz=0 0 0.05 rpy=0 0 0 -> xyz=0.0 0.0 0.2 rpy=0 -1.57 0
- joint eef_joint: axis 1 0 0 -> 0 1 0; origin xyz=0 0 0.0 rpy=0 0 0 -> xyz=0 0.3 0.0 rpy=0 0 0
- joint el_joint: axis 0 0 1 -> 1 0 0; origin xyz=0 0 0.05 rpy=1.57 0 0 -> xyz=-0.05 -0.05 0.04 rpy=1.57 1.57 0; parent azimuth_link -> azimuth_servo
